Commit message: the gripper added

File: src/arm_sim/urdf/arm.urdf.xacro (robot description, xacro)
@@ -15,4 +15,7 @@
     <color rgba="0.0 1.0 0.0 1.0"/>
   </material>
+  <material name="yellow">
+    <color rgba="1.0 1.0 0.0 1.0"/>
+  </material>
   <!-- ===== WORLD + FIXED BASE ===== -->
   <link name="world"/>
@@ -129,4 +132,34 @@
     <child link="link3"/>
     <origin xyz="0 0 0.061" rpy="0 0 0"/>
+    <axis xyz="0 1 0"/>
+    <limit lower="${-pi/2}" upper="${pi/2}" effort="10.0" velocity="1.0"/>
+    <dynamics damping="0.1" friction="0.1"/>
+  </joint>
+  <!-- ===== gripper ===== -->
+  <link name="gripper">
+    <inertial>
+      <origin xyz="-0.01 -0.013 -0.01" rpy="0 0 0"/>
+      <mass value="1"/>
+      <inertia ixx="0.0333" ixy="0.0" ixz="0.0" iyy="0.0333" iyz="0.0" izz="0.006667"/>
+    </inertial>
+    <visual>
+      <origin xyz="-0.01 -0.013 -0.01" rpy="0 0 0"/>
+      <geometry>
+        <mesh filename="package://arm_sim/meshes/gripper.STL" scale="0.001 0.001 0.001"/>
+      </geometry>
+      <material name="green"/>
+    </visual>
+    <collision>
+      <origin xyz="-0.01 -0.013 -0.01" rpy="0 0 0"/>
+      <geometry>
+        <mesh filename="package://arm_sim/meshes/gripper.STL" scale="0.001 0.001 0.001"/>
+      </geometry>
+    </collision>
+  </link>
+  <!-- THIRD joint: REVOLUTE -->
+  <joint name="gripper_joint" type="revolute">
+    <parent link="link3"/>
+    <child link="gripper"/>
+    <origin xyz="0 0 0.061" rpy="0 ${-pi/2} 0"/>
     <axis xyz="0 1 0"/>
     <limit lower="${-pi/2}" upper="${pi/2}" effort="10.0" velocity="1.0"/>
@@ -165,4 +198,13 @@
       <state_interface name="effort"/>
     </joint>
+    <joint name="gripper_joint">
+      <command_interface name="position">
+        <param name="min">${-pi/2}</param>
+        <param name="max">${pi/2}</param>
+      </command_interface>
+      <state_interface name="position"/>
+      <state_interface name="velocity"/>
+      <state_interface name="effort"/>
+    </joint>
   </ros2_control>
   <!-- ===== Gazebo plugin: starts controller_manager, loads the yaml ===== -->
@@ -185,3 +227,6 @@
     <material>Gazebo/Green</material>
   </gazebo>
+  <gazebo reference="gripper">
+    <material>Gazebo/Yellow</material>
+  </gazebo>
 </robot>

Commit message: update

File: src/arm_sim/urdf/arm.urdf.xacro (robot description, xacro)
@@ -1,170 +1,481 @@
-<?xml version="1.0"?>
-<robot xmlns:xacro="http://www.ros.org/wiki/xacro" name="three_link_arm">
-  <xacro:property name="pi" value="3.14159265359"/>
-  <!-- ===== MATERIALS (for RViz) ===== -->
-  <material name="gray">
-    <color rgba="0.5 0.5 0.5 1.0"/>
-  </material>
-  <material name="blue">
-    <color rgba="0.0 0.0 1.0 1.0"/>
-  </material>
-  <material name="red">
-    <color rgba="1.0 0.0 0.0 1.0"/>
-  </material>
-  <material name="green">
-    <color rgba="0.0 1.0 0.0 1.0"/>
-  </material>
-  <material name="yellow">
-    <color rgba="1.0 1.0 0.0 1.0"/>
-  </material>
-  <!-- ===== WORLD + FIXED BASE ===== -->
+<?xml version="1.0" encoding="utf-8"?>
+<!-- This URDF was automatically created by SolidWorks to URDF Exporter! Originally created by Stephen Brawner (brawner@gmail.com)
+     Commit Version: 1.5.1-0-g916b5db  Build Version: 1.5.7152.31018
+     For more information, please see http://wiki.ros.org/sw_urdf_exporter -->
+<robot name="arm" xmlns:xacro="http://www.ros.org/wiki/xacro">
   <link name="world"/>
-    <link name="base_link">
-    <inertial>
-      <origin xyz="0 0 0" rpy="${pi/2} 0 ${pi/2}"/>
-      <mass value="5.0"/>
-      <inertia ixx="0.1" ixy="0.0" ixz="0.0" iyy="0.1" iyz="0.0" izz="0.1"/>
-    </inertial>
-    <visual>
-      <origin xyz="0 0 0" rpy="${pi/2} 0 ${pi/2}"/>
-      <geometry>
-        <mesh filename="package://arm_sim/meshes/base.STL" scale="0.001 0.001 0.001"/>
-      </geometry>
-      <material name="gray"/>
-    </visual>
-    <collision>
-      <origin xyz="0 0 0" rpy="${pi/2} 0 ${pi/2}"/>
-      <geometry>
-        <mesh filename="package://arm_sim/meshes/base.STL" scale="0.001 0.001 0.001"/>
-      </geometry>
-    </collision>
-  </link>
-  <!-- FIRST joint: fixed (anchors base to the world) -->
+  <link
+    name="base_link">
+    <inertial>
+      <origin
+        xyz="-1.0639E-18 0 0.0225"
+        rpy="0 0 0" />
+      <mass
+        value="0.05768" />
+      <inertia
+        ixx="1.5501E-05"
+        ixy="0"
+        ixz="-1.9481E-37"
+        iyy="1.5501E-05"
+        iyz="-5.0159E-38"
+        izz="1.1536E-05" />
+    </inertial>
+    <visual>
+      <origin
+        xyz="0 0 0"
+        rpy="0 0 0" />
+      <geometry>
+        <mesh
+          filename="package://arm_sim/meshes/base_link.STL" />
+      </geometry>
+      <material
+        name="">
+        <color
+          rgba="1 1 1 1" />
+      </material>
+    </visual>
+    <collision>
+      <origin
+        xyz="0 0 0"
+        rpy="0 0 0" />
+      <geometry>
+        <mesh
+          filename="package://arm_sim/meshes/base_link.STL" />
+      </geometry>
+    </collision>
+  </link>
   <joint name="world_to_base" type="fixed">
     <parent link="world"/>
     <child link="base_link"/>
-    <origin xyz="-0.05 -0.05 0" rpy="0 0 0"/>
-  </joint>
-  <!-- ===== LINK 1 ===== -->
-  <link name="link1">
-    <inertial>
-      <origin xyz="-0.01 -0.013 -0.01" rpy="0 0 0"/>
-      <mass value="1.5"/>
-      <inertia ixx="0.05" ixy="0.0" ixz="0.0" iyy="0.05" iyz="0.0" izz="0.01"/>
-    </inertial>
-    <visual>
-      <origin xyz="-0.01 -0.013 -0.01" rpy="0 0 0"/>
-      <geometry>
-        <mesh filename="package://arm_sim/meshes/link.STL" scale="0.001 0.001 0.001"/>
-      </geometry>
-      <material name="blue"/>
-    </visual>
-    <collision>
-      <origin xyz="-0.01 -0.013 -0.01" rpy="0 0 0"/>
-      <geometry>
-        <mesh filename="package://arm_sim/meshes/link.STL" scale="0.001 0.001 0.001"/>
-      </geometry>
-    </collision>
-  </link>
-  <!-- SECOND joint: REVOLUTE -->
-  <joint name="joint1" type="revolute">
-    <parent link="base_link"/>
-    <child link="link1"/>
-    <origin xyz="0.05 0.05 0.061" rpy="0 0 0"/>
-    <axis xyz="0 1 0"/>
-    <limit lower="${-pi/2}" upper="${pi/2}" effort="10.0" velocity="1.0"/>
-    <dynamics damping="0.1" friction="0.1"/>
-  </joint>
-  <!-- ===== LINK 2 ===== -->
-  <link name="link2">
-    <inertial>
-      <origin xyz="-0.01 -0.013 -0.01" rpy="0 0 0"/>
-      <mass value="1.5"/>
-      <inertia ixx="0.05" ixy="0.0" ixz="0.0" iyy="0.05" iyz="0.0" izz="0.01"/>
-    </inertial>
-    <visual>
-      <origin xyz="-0.01 -0.013 -0.01" rpy="0 0 0"/>
-      <geometry>
-        <mesh filename="package://arm_sim/meshes/link.STL" scale="0.001 0.001 0.001"/>
-      </geometry>
-      <material name="red"/>
-    </visual>
-    <collision>
-      <origin xyz="-0.01 -0.013 -0.01" rpy="0 0 0"/>
-      <geometry>
-        <mesh filename="package://arm_sim/meshes/link.STL" scale="0.001 0.001 0.001"/>
-      </geometry>
-    </collision>
-  </link>
-  <!-- THIRD joint: REVOLUTE -->
-  <joint name="joint2" type="revolute">
-    <parent link="link1"/>
-    <child link="link2"/>
-    <origin xyz="0 0 0.061" rpy="0 0 0"/>
-    <axis xyz="0 1 0"/>
-    <limit lower="${-pi/2}" upper="${pi/2}" effort="10.0" velocity="1.0"/>
-    <dynamics damping="0.1" friction="0.1"/>
-  </joint>
-  <!-- ===== LINK 3 ===== -->
-  <link name="link3">
-    <inertial>
-      <origin xyz="-0.01 -0.013 -0.01" rpy="0 0 0"/>
-      <mass value="1.5"/>
-      <inertia ixx="0.05" ixy="0.0" ixz="0.0" iyy="0.05" iyz="0.0" izz="0.01"/>
-    </inertial>
-    <visual>
-      <origin xyz="-0.01 -0.013 -0.01" rpy="0 0 0"/>
-      <geometry>
-        <mesh filename="package://arm_sim/meshes/link.STL" scale="0.001 0.001 0.001"/>
-      </geometry>
-      <material name="green"/>
-    </visual>
-    <collision>
-      <origin xyz="-0.01 -0.013 -0.01" rpy="0 0 0"/>
-      <geometry>
-        <mesh filename="package://arm_sim/meshes/link.STL" scale="0.001 0.001 0.001"/>
-      </geometry>
-    </collision>
-  </link>
-  <!-- THIRD joint: REVOLUTE -->
-  <joint name="joint3" type="revolute">
-    <parent link="link2"/>
-    <child link="link3"/>
-    <origin xyz="0 0 0.061" rpy="0 0 0"/>
-    <axis xyz="0 1 0"/>
-    <limit lower="${-pi/2}" upper="${pi/2}" effort="10.0" velocity="1.0"/>
-    <dynamics damping="0.1" friction="0.1"/>
-  </joint>
-  <!-- ===== gripper ===== -->
-  <link name="gripper">
-    <inertial>
-      <origin xyz="-0.01 -0.013 -0.01" rpy="0 0 0"/>
-      <mass value="1"/>
-      <inertia ixx="0.0333" ixy="0.0" ixz="0.0" iyy="0.0333" iyz="0.0" izz="0.006667"/>
-    </inertial>
-    <visual>
-      <origin xyz="-0.01 -0.013 -0.01" rpy="0 0 0"/>
-      <geometry>
-        <mesh filename="package://arm_sim/meshes/gripper.STL" scale="0.001 0.001 0.001"/>
-      </geometry>
-      <material name="green"/>
-    </visual>
-    <collision>
-      <origin xyz="-0.01 -0.013 -0.01" rpy="0 0 0"/>
-      <geometry>
-        <mesh filename="package://arm_sim/meshes/gripper.STL" scale="0.001 0.001 0.001"/>
-      </geometry>
-    </collision>
-  </link>
-  <!-- THIRD joint: REVOLUTE -->
-  <joint name="gripper_joint" type="revolute">
-    <parent link="link3"/>
-    <child link="gripper"/>
-    <origin xyz="0 0 0.061" rpy="0 ${-pi/2} 0"/>
-    <axis xyz="0 1 0"/>
-    <limit lower="${-pi/2}" upper="${pi/2}" effort="10.0" velocity="1.0"/>
-    <dynamics damping="0.1" friction="0.1"/>
-  </joint>
-  <!-- ===== ros2_control: declares joint's interfaces ===== -->
+    <origin xyz="0 0 0" rpy="0 0 0"/>
+  </joint>
+  <link
+    name="link1">
+    <inertial>
+      <origin
+        xyz="-4.0978E-19 -9.8755E-18 0.0025911"
+        rpy="0 0 0" />
+      <mass
+        value="0.0086396" />
+      <inertia
+        ixx="1.0316E-06"
+        ixy="-1.4108E-23"
+        ixz="1.4E-23"
+        iyy="1.2174E-06"
+        iyz="-1.4338E-21"
+        izz="1.6687E-06" />
+    </inertial>
+    <visual>
+      <origin
+        xyz="0 0 0"
+        rpy="0 0 0" />
+      <geometry>
+        <mesh
+          filename="package://arm_sim/meshes/link1.STL" />
+      </geometry>
+      <material
+        name="">
+        <color
+          rgba="1 1 1 0.32" />
+      </material>
+    </visual>
+    <collision>
+      <origin
+        xyz="0 0 0"
+        rpy="0 0 0" />
+      <geometry>
+        <mesh
+          filename="package://arm_sim/meshes/link1.STL" />
+      </geometry>
+    </collision>
+  </link>
+  <joint
+    name="joint1"
+    type="revolute">
+    <origin
+      xyz="0 0 0.0475"
+      rpy="0 0 0" />
+    <parent
+      link="base_link" />
+    <child
+      link="link1" />
+    <axis
+      xyz="0 0 -1" />
+    <limit
+      lower="-1.57"
+      upper="1.57"
+      effort="10"
+      velocity="1" />
+    <dynamics
+      damping="0.1"
+      friction="0.1" />
+  </joint>
+  <link
+    name="link2">
+    <inertial>
+      <origin
+        xyz="-0.026754 -0.00028438 2.3123E-19"
+        rpy="0 0 0" />
+      <mass
+        value="0.014541" />
+      <inertia
+        ixx="1.2234E-06"
+        ixy="-2.0157E-08"
+        ixz="1.9988E-22"
+        iyy="3.1196E-06"
+        iyz="6.8418E-23"
+        izz="2.8107E-06" />
+    </inertial>
+    <visual>
+      <origin
+        xyz="0 0 0"
+        rpy="0 0 0" />
+      <geometry>
+        <mesh
+          filename="package://arm_sim/meshes/link2.STL" />
+      </geometry>
+      <material
+        name="">
+        <color
+          rgba="1 1 1 1" />
+      </material>
+    </visual>
+    <collision>
+      <origin
+        xyz="0 0 0"
+        rpy="0 0 0" />
+      <geometry>
+        <mesh
+          filename="package://arm_sim/meshes/link2.STL" />
+      </geometry>
+    </collision>
+  </link>
+  <joint
+    name="joint2"
+    type="revolute">
+    <origin
+      xyz="0 0 0.0135"
+      rpy="0 1.5708 0" />
+    <parent
+      link="link1" />
+    <child
+      link="link2" />
+    <axis
+      xyz="0 0 -1" />
+    <limit
+      lower="-1.57"
+      upper="1.57"
+      effort="10"
+      velocity="1" />
+    <dynamics
+      damping="0.1"
+      friction="0.1" />
+  </joint>
+  <link
+    name="link3">
+    <inertial>
+      <origin
+        xyz="-0.026754 -0.00028438 5.7937E-19"
+        rpy="0 0 0" />
+      <mass
+        value="0.014541" />
+      <inertia
+        ixx="1.2234E-06"
+        ixy="-2.0157E-08"
+        ixz="2.811E-22"
+        iyy="3.1196E-06"
+        iyz="-6.1017E-23"
+        izz="2.8107E-06" />
+    </inertial>
+    <visual>
+      <origin
+        xyz="0 0 0"
+        rpy="0 0 0" />
+      <geometry>
+        <mesh
+          filename="package://arm_sim/meshes/link3.STL" />
+      </geometry>
+      <material
+        name="">
+        <color
+          rgba="1 1 1 1" />
+      </material>
+    </visual>
+    <collision>
+      <origin
+        xyz="0 0 0"
+        rpy="0 0 0" />
+      <geometry>
+        <mesh
+          filename="package://arm_sim/meshes/link3.STL" />
+      </geometry>
+    </collision>
+  </link>
+  <joint
+    name="joint3"
+    type="revolute">
+    <origin
+      xyz="-0.060997 -0.00064835 0"
+      rpy="0 0 0" />
+    <parent
+      link="link2" />
+    <child
+      link="link3" />
+    <axis
+      xyz="0 0 -1" />
+    <limit
+      lower="-1.57"
+      upper="1.57"
+      effort="10"
+      velocity="1" />
+    <dynamics
+      damping="0.1"
+      friction="0.1" />
+  </joint>
+  <link
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